File: pcb/bancouver40_cfx/bancouver40_cfx.kicad_pcb (KiCad board)
At the start: 2 copper layers, 170 x 68 mm, 83 parts, among them J1 Conn_01x02_Female, J2 Conn_01x02_Female, SW1 SW_Push, SW10 SW_Push, SW11 SW_Push, SW12 SW_Push, SW13 SW_Push, SW14 SW_Push, SW15 SW_Push, SW16 SW_Push, SW17 SW_Push, SW18 SW_Push, SW19 SW_Push, SW2 SW_Push, SW20 SW_Push, SW21 SW_Push, SW22 SW_Push, SW23 SW_Push, SW24 SW_Push, SW25 SW_Push, SW26 SW_Push, SW27 SW_Push, SW28 SW_Push, SW29 SW_Push, SW3 SW_Push, SW30 SW_Push, SW33 SW_Push, SW34 SW_Push, SW35 SW_Push, SW36 SW_Push, SW37 SW_Push, SW38 SW_Push, SW4 SW_Push, SW41 SW_SPST, SW5 SW_Push, SW6 SW_Push, SW7 SW_Push, SW8 SW_Push, SW9 SW_Push, U1 xiao-ble, U2 74HC595

Commit message: add cnc files
Other:
- board text added: "babbit36 by sporewoh v1.0"
- board text added: "off"
- board text added: "on"
- board text removed: "babbit36 by sporewoh v0.0"
